File: KiCad/Capacitor_Bank.kicad_pcb (KiCad board)
At the start: 2 copper layers, 78.5 x 67.5 mm, 42 parts, among them J1 Conn_01x02, SW1 SW_DIP_x09, SW2 SW_DIP_x09, SW3 SW_DIP_x09, SW4 SW_DIP_x09

Commit message: Add files via upload
Parts:
- C1, C2, C3, C4, C5, C6, C7, C8, C9: footprint Capacitor_THT:C_Disc_D3.8mm_W2.6mm_P2.50mm -> Capacitor_THT:C_Disc_D4.7mm_W2.5mm_P5.00mm
- moved C2 4.45 mm to (166.3, 40.1)
- moved C4 4.45 mm to (166.3, 45.2)
- moved C6 4.45 mm to (166.3, 50.6)
- moved C8 4.45 mm to (166.3, 55.4)
- moved C1 1.91 mm to (159.0, 37.4)
- moved C3 1.91 mm to (159.1, 42.7)
- moved C5 1.91 mm to (159.1, 48.1)
- moved C7 1.91 mm to (159.1, 52.9)
- moved C9 1.91 mm to (159.1, 57.8)
Routing:
- net Net-(J1-Pin_2): track 311.4 -> 308.7 mm
- net Net-(C6-Pad2): track 8.31 -> 10.3 mm
- net Net-(C8-Pad2): track 8.22 -> 10.2 mm
- net Net-(C4-Pad2): track 8.20 -> 10.1 mm
- net Net-(C2-Pad2): track 8.19 -> 10.1 mm
- net Net-(C9-Pad2): track 3.39 -> 2.79 mm
- net Net-(C7-Pad2): track 3.48 -> 2.89 mm
- net Net-(C5-Pad2): track 3.58 -> 2.98 mm
- net Net-(C3-Pad2): track 3.47 -> 2.87 mm
- net Net-(C1-Pad2): track 3.33 -> 2.73 mm
